File: board-b-sensor/board-b-sensor.kicad_sch (KiCad schematic)
At the start: 0 parts

Commit message: session-1: board-b schematic complete, ERC clean
All sensor components placed and wired: MAX30102 (HR/SpO2), MAX30208
(skin temp, I2C addr 0x50), AD8232 (ECG, unity-gain feedback on
OPAMP-), ADS1115 (4-ch ADC). Decoupling caps, I2C pull-ups, and
PWR_FLAG symbols added. Fixed MAX30208 lib_symbols sub-symbol format
for KiCAD 10 SWIG parser compatibility. ERC result: 0 errors, 79
acceptable warnings (AD8232 off-grid pins, custom footprint lib).

Co-Authored-By: Claude Sonnet 4.6 <noreply@anthropic.com>
Parts:
- added C_ADC, C_HP1, C_HP2, C_LED2, C_M3V, C_T1, C_VS: 100nF, Capacitor_SMD:C_0402_1005Metric, symbol Device:C
- added C_LED1: 10uF, Capacitor_SMD:C_0805_2012Metric, symbol Device:C
- added C_OP: 10nF, Capacitor_SMD:C_0402_1005Metric, symbol Device:C
- added D1, D2: BAV99, Package_TO_SOT_SMD:SOT-23, symbol Diode:BAV99
- added J1: FPC_INTER_BOARD, Connector_FFC-FPC:Hirose_FH12-10S-0.5SH_1x10-1MP_P0.50mm_Horizontal, symbol Connector_Generic:Conn_01x10
- added J_GSRN: POGO_GSR_N, custom:Pogo_P75B1_TH, symbol Connector_Generic:Conn_01x01
- added J_GSRP: POGO_GSR_P, custom:Pogo_P75B1_TH, symbol Connector_Generic:Conn_01x01
- added J_LA: POGO_ECG_LA, custom:Pogo_P75B1_TH, symbol Connector_Generic:Conn_01x01
- added J_RA: POGO_ECG_RA, custom:Pogo_P75B1_TH, symbol Connector_Generic:Conn_01x01
- added R_GAIN: 200k, Resistor_SMD:R_0402_1005Metric, symbol Device:R
- added R_GSR1, R_GSR2, R_GSRREF: 10k, Resistor_SMD:R_0402_1005Metric, symbol Device:R
- added R_HP1, R_HP2: 300k, Resistor_SMD:R_0402_1005Metric, symbol Device:R
- added R_LA, R_OP, R_RA, R_RL: 100k, Resistor_SMD:R_0402_1005Metric, symbol Device:R
- added R_SCL, R_SDA: 4.7k, Resistor_SMD:R_0402_1005Metric, symbol Device:R
- added U1: MAX30102, custom:MAX30102EFDT, symbol MAX30102:MAX30102EFD_T
- added U2: MAX30208, custom:MAX30208CLBT, symbol MAX30208:MAX30208CLB+T
- added U3: AD8232, Package_DFN_QFN:QFN-10-1EP_2x2mm_P0.5mm_EP0.6x0.6mm, symbol AD8232:AD8232ACPZ-R7
- added U4: ADS1115, Package_VSSOP:VSSOP-10_3x3mm_P0.5mm, symbol Analog_ADC:ADS1115IDGS
Connections:
- new net AD8232_SDN: J1.6 (Pin_6), U3.13 (SDN)
- new net AGND: C_ADC.2, C_HP1.2, C_HP2.2, C_OP.2, C_VS.2, U3.14 (AC/DC), U3.15 (FR), U3.16 (GND), U4.1 (ADDR), U4.3 (GND)
- new net ECG_LA: D2.2 (A), J_LA.1 (Pin_1), R_LA.1
- new net ECG_LA_F: R_HP1.2, R_LA.2, U3.2 (+IN)
- new net ECG_OUT: U3.10 (OUT), U4.4 (AIN0)
- new net ECG_RA: D1.2 (A), J_RA.1 (Pin_1), R_RA.1
- new net ECG_RA_F: R_HP2.2, R_RA.2, U3.3 (-IN)
- new net GAIN_A: R_GAIN.1, R_OP.1, U3.19 (IAOUT)
- new net GAIN_B: R_GAIN.2, U3.18 (REFIN), U3.8 (REFOUT)
- new net GND: C_LED1.2, C_LED2.2, C_M3V.2, C_T1.2, D1.3 (K), D2.3 (K), J1.2 (Pin_2), J1.3 (Pin_3), U1.12 (GND), U1.4 (PGND), U2.10 (GPIO0), U2.4 (GND_1), U2.5 (GND_2), U2.6 (GND_3), U2.7 (GPIO1)
- new net GSR_H: R_GSR1.2, R_GSRREF.2, U4.5 (AIN1)
- new net GSR_L: R_GSR2.2, U4.6 (AIN2)
- new net GSR_N: J_GSRN.1 (Pin_1), R_GSR2.1
- new net GSR_P: J_GSRP.1 (Pin_1), R_GSR1.1
- new net HP_N1: C_HP2.1, R_HP2.1, U3.1 (HPDRIVE)
- new net HP_P1: C_HP1.1, R_HP1.1, U3.20 (HPSENSE)
- new net LO_MINUS: J1.7 (Pin_7), U3.11 (LOD-)
- new net LO_PLUS: J1.8 (Pin_8), U3.12 (LOD+)
- new net OP_AM: U3.6 (SW), U3.9 (OPAMP-)
- new net OP_AP: C_OP.1, R_OP.2, U3.7 (OPAMP+)
- new net RLDRIVE: J1.9 (Pin_9), R_RL.2, U3.4 (RLDFB)
- new net RLDRIVE_IC: R_RL.1, U3.5 (RLD)
- new net SCL: J1.5 (Pin_5), R_SCL.2, U1.2 (SCL), U2.9 (SCL), U4.10 (SCL)
- new net SDA: J1.4 (Pin_4), R_SDA.2, U1.3 (SDA), U2.8 (SDA), U4.9 (SDA)
- new net VCC_3V3: C_ADC.1, C_LED1.1, C_LED2.1, C_M3V.1, C_T1.1, C_VS.1, D1.1 (K), D2.1 (K), J1.1 (Pin_1), R_GSRREF.1, R_SCL.1, R_SDA.1, U1.10 (VLED+), U1.11 (VDD), U1.9 (VLED+), U2.1 (VDD_1), U2.2 (VDD_2), U2.3 (VDD_3), U3.17 (+VS), U4.8 (VDD)
- no-connect marks 0 -> 4
Changed lines of the file:
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@@
-(kicad_sch (version 20250114) (generator "KiCAD-MCP-Server")
-  (paper "A4")
-  (sheet_instances
-    (path "/" (page "1"))
-  )
-)
