File: board-b-sensor/board-b-sensor.kicad_sch (KiCad schematic)
At the start: 32 parts, among them J1 FPC_INTER_BOARD, U1 MAX30102, U2 MAX30208, U3 AD8232, U4 ADS1115

Commit message: session-1/2: board-b schematic + PCB progress, update gitignore
Parts:
- U3: footprint Package_DFN_QFN:QFN-10-1EP_2x2mm_P0.5mm_EP0.6x0.6mm -> Package_DFN_QFN:QFN-20-1EP_4x4mm_P0.5mm_EP2.6x2.6mm
