File: board-b-sensor/board-b-sensor.kicad_sch (KiCad schematic)
At the start: 32 parts, among them J1 FPC_INTER_BOARD, U1 MAX30102, U2 MAX30208, U3 AD8232, U4 ADS1115

Commit message: session-2: board-a progress + board-b schematic updates
Co-Authored-By: Claude Sonnet 4.6 <noreply@anthropic.com>
Parts:
- removed C_ADC, C_HP1, C_HP2, C_LED2, C_M3V, C_T1, C_VS: 100nF, Capacitor_SMD:C_0402_1005Metric, symbol Device:C
- removed C_LED1: 10uF, Capacitor_SMD:C_0805_2012Metric, symbol Device:C
- removed C_OP: 10nF, Capacitor_SMD:C_0402_1005Metric, symbol Device:C
- removed D1, D2: BAV99, Package_TO_SOT_SMD:SOT-23, symbol Diode:BAV99
- removed J1: FPC_INTER_BOARD, Connector_FFC-FPC:Hirose_FH12-10S-0.5SH_1x10-1MP_P0.50mm_Horizontal, symbol Connector_Generic:Conn_01x10
- removed J_GSRN: POGO_GSR_N, custom:Pogo_P75B1_TH, symbol Connector_Generic:Conn_01x01
- removed J_GSRP: POGO_GSR_P, custom:Pogo_P75B1_TH, symbol Connector_Generic:Conn_01x01
- removed J_LA: POGO_ECG_LA, custom:Pogo_P75B1_TH, symbol Connector_Generic:Conn_01x01
- removed J_RA: POGO_ECG_RA, custom:Pogo_P75B1_TH, symbol Connector_Generic:Conn_01x01
- removed R_GAIN: 200k, Resistor_SMD:R_0402_1005Metric, symbol Device:R
- removed R_GSR1, R_GSR2, R_GSRREF: 10k, Resistor_SMD:R_0402_1005Metric, symbol Device:R
- removed R_HP1, R_HP2: 300k, Resistor_SMD:R_0402_1005Metric, symbol Device:R
- removed R_LA, R_OP, R_RA, R_RL: 100k, Resistor_SMD:R_0402_1005Metric, symbol Device:R
- removed R_SCL, R_SDA: 4.7k, Resistor_SMD:R_0402_1005Metric, symbol Device:R
- removed U1: MAX30102, custom:MAX30102EFDT, symbol MAX30102:MAX30102EFD_T
- removed U2: MAX30208, custom:MAX30208CLBT, symbol MAX30208:MAX30208CLB+T
- removed U3: AD8232, Package_DFN_QFN:QFN-20-1EP_4x4mm_P0.5mm_EP2.6x2.6mm, symbol AD8232:AD8232ACPZ-R7
- removed U4: ADS1115, Package_VSSOP:VSSOP-10_3x3mm_P0.5mm, symbol Analog_ADC:ADS1115IDGS
Connections:
- no-connect marks 4 -> 0
Changed lines of the file:
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@@
+(kicad_sch
+	(version 20260306)
+	(generator "eeschema")
+	(generator_version "10.0")
+	(paper "A4")
+	(sheet_instances
+		(path "/"
+			(page "1")
+		)
+	)
+	(embedded_fonts no)
+)

Commit message: feat: add Board B sensor schematic and initial PCB layout
Schematic includes MAX30208, AD8232, ADS1115, MAX30102 with AP2112K-1.8V LDO and BSS138 level shifters for I2C. PCB layout started with component placement on 25x25mm board.

Co-Authored-By: Claude Sonnet 4.6 <noreply@anthropic.com>
Parts:
- added C1, C2, C3, C4, C5, C7, C9, C_LDO_OUT2: 100nF, Capacitor_SMD:C_0402_1005Metric, symbol Device:C
- added C8, C_LDO_IN1, C_LDO_OUT1: 10uF, Capacitor_SMD:C_0805_2012Metric, symbol Device:C
- added IC1: MAX30208CLB+T, custom:MAX30208CLBT, symbol MAX30208CLB+T:MAX30208CLB+T
- added J1: Conn_01x10_Socket, 1_Global_Library:FPC-SMD_10P-P0.50_XUNPU_FPC-05F-10PH15, symbol Connector:Conn_01x10_Socket
- added J_GSR+1, J_GSR-1, J_LA1, J_RA1: Conn_01x01, TestPoint:TestPoint_Pad_D2.0mm, symbol Connector_Generic:Conn_01x01
- added Q1, Q2, Q3: BSS138, Package_TO_SOT_SMD:SOT-23, symbol Transistor_FET:BSS138
- added R1, R2, R3: 100k, Resistor_SMD:R_0402_1005Metric, symbol Device:R
- added R10, R11, R12, R13, R14, R9: 4.7k, Resistor_SMD:R_0402_1005Metric, symbol Device:R
- added R15, R5, R6, R7, R8: 10k, Resistor_SMD:R_0402_1005Metric, symbol Device:R
- added R4: 300k, Resistor_SMD:R_0402_1005Metric, symbol Device:R
- added U1: AD8232ACPZ-R7, Package_DFN_QFN:QFN-20-1EP_4x4mm_P0.5mm_EP2.6x2.6mm, symbol AD8232ACPZ-R7:AD8232ACPZ-R7
- added U2: ADS1115IDGS, Package_SO:TSSOP-10_3x3mm_P0.5mm, symbol Analog_ADC:ADS1115IDGS
- added U3: MAX30102, OptoDevice:Maxim_OLGA-14_3.3x5.6mm_P0.8mm, symbol Sensor:MAX30102
- added U4: AP2112K-1.8, Package_TO_SOT_SMD:SOT-23-5, symbol Regulator_Linear:AP2112K-1.8
Connections:
- new net: C_LDO_OUT1.1, C_LDO_OUT2.2, U4.5 (VOUT)
- new net: R4.1, U1.1 (HPDRIVE)
- new net: C3.1, U1.18 (REFIN), U1.4 (RLDFB), U1.7 (OPAMP+), U1.8 (REFOUT)
- new net: R1.2, U1.2 (+IN)
- new net: C4.2, R4.2, U1.20 (HPSENSE)
- new net: R2.1, U1.3 (-IN)
- new net: R3.1, U1.5 (RLD)
- new net: R6.2, R7.2, U2.6 (AIN2)
- new net: R5.2, R8.2, U2.5 (AIN1)
- new net +1V8: C9.2, C_LDO_OUT1.2, C_LDO_OUT2.1, Q1.1 (G), Q2.1 (G), Q3.1 (G), R10.2, R12.2, R14.2, U3.11 (VDD)
- new net +3.3V: C1.1, C2.2, C5.2, C7.1, C8.1, C_LDO_IN1.2, IC1.1 (VDD_1), IC1.2 (VDD_2), IC1.3 (VDD_3), J1.1 (Pin_1), R11.1, R13.1, R15.2, R8.1, R9.1, U1.14 (AC/DC), U1.17 (+VS), U2.8 (VDD), U3.10 (VLED+), U3.9 (VLED+), U4.1 (VIN), U4.3 (EN)
- new net ECG_LOD+: J1.8 (Pin_8), U1.12 (LOD+)
- new net ECG_LOD-: J1.7 (Pin_7), U1.11 (LOD-)
- new net ECG_OUT: U1.10 (OUT), U1.9 (OPAMP-), U2.4 (AIN0)
- new net ECG_RLD_PAD: J1.9 (Pin_9), R3.2
- new net ECG_SDN: J1.6 (Pin_6), U1.13 (SDN)
- new net GND: C1.2, C2.1, C3.2, C4.1, C5.1, C7.2, C8.2, C9.1, C_LDO_IN1.1, IC1.4 (GND_1), IC1.5 (GND_2), IC1.6 (GND_3), J1.2 (Pin_2), R6.1, U1.15 (FR), U1.16 (GND), U2.1 (ADDR), U2.3 (GND), U3.12 (GND), U3.4 (PGND), U4.2 (GND)
- new net GSR+: J_GSR+1.1 (Pin_1), R5.1
- new net GSR-: J_GSR-1.1 (Pin_1), R7.1
- new net INT_ADC: J1.3 (Pin_3), R15.1, U2.2 (ALERT/RDY)
- new net INT_MAX: J1.10 (Pin_10), Q3.3 (D), R13.2
- new net INT_MAX_1V8: Q3.2 (S), R14.1, U3.13 (~{INT})
- new net LA: J_LA1.1 (Pin_1), R1.1
- new net RA: J_RA1.1 (Pin_1), R2.2
- new net SCL: IC1.9 (SCL), J1.5 (Pin_5), Q2.3 (D), R11.2, U2.10 (SCL)
- new net SCL_1V8: Q2.2 (S), R12.1, U3.2 (SCL)
- new net SDA: IC1.8 (SDA), J1.4 (Pin_4), Q1.3 (D), R9.2, U2.9 (SDA)
- new net SDA_1V8: Q1.2 (S), R10.1, U3.3 (SDA)
- no-connect marks 0 -> 5
