File: board-b-sensor/board-b-sensor.kicad_pcb (KiCad board)
At the start: 2 copper layers, 0 parts

Commit message: session-1/2: board-b schematic + PCB progress, update gitignore
Parts:
- added C_ADC: 100nF, Capacitor_SMD:C_0402_1005Metric, F.Cu at (21.0, 16.0)
- added C_HP1: 100nF, Capacitor_SMD:C_0402_1005Metric, F.Cu at (1.50, 14.0)
- added C_HP2: 100nF, Capacitor_SMD:C_0402_1005Metric, F.Cu at (1.50, 15.5)
- added C_LED1: 10uF, Capacitor_SMD:C_0805_2012Metric, B.Cu at (4.50, 13.5)
- added C_LED2: 100nF, Capacitor_SMD:C_0402_1005Metric, B.Cu at (8.00, 13.5)
- added C_M3V: 100nF, Capacitor_SMD:C_0402_1005Metric, B.Cu at (10.0, 13.5)
- added C_OP: 10nF, Capacitor_SMD:C_0402_1005Metric, F.Cu at (9.50, 9.50)
- added C_T1: 100nF, Capacitor_SMD:C_0402_1005Metric, B.Cu at (17.0, 13.5)
- added C_VS: 100nF, Capacitor_SMD:C_0402_1005Metric, F.Cu at (11.0, 12.0)
- added D1: BAV99, Package_TO_SOT_SMD:SOT-23, F.Cu at (4.00, 19.5)
- added D2: BAV99, Package_TO_SOT_SMD:SOT-23, F.Cu at (10.0, 19.5)
- added J1: FPC_INTER_BOARD, Connector_FFC-FPC:Hirose_FH12-10S-0.5SH_1x10-1MP_P0.50mm_Horizontal, F.Cu at (12.5, 6.45)
- added J_GSRN: POGO_GSR_N, custom:Pogo_P75B1_TH, F.Cu at (22.0, 23.5)
- added J_GSRP: POGO_GSR_P, custom:Pogo_P75B1_TH, F.Cu at (16.0, 23.5)
- added J_LA: POGO_ECG_LA, custom:Pogo_P75B1_TH, F.Cu at (10.0, 23.5)
- added J_RA: POGO_ECG_RA, custom:Pogo_P75B1_TH, F.Cu at (4.00, 23.5)
- added R_GAIN: 200k, Resistor_SMD:R_0402_1005Metric, F.Cu at (7.00, 12.0)
- added R_GSR1: 10k, Resistor_SMD:R_0402_1005Metric, F.Cu at (22.0, 16.0)
- added R_GSR2: 10k, Resistor_SMD:R_0402_1005Metric, F.Cu at (22.0, 18.0)
- added R_GSRREF: 10k, Resistor_SMD:R_0402_1005Metric, F.Cu at (22.0, 14.0)
- added R_HP1: 300k, Resistor_SMD:R_0402_1005Metric, F.Cu at (3.00, 14.0)
- added R_HP2: 300k, Resistor_SMD:R_0402_1005Metric, F.Cu at (3.00, 15.5)
- added R_LA: 100k, Resistor_SMD:R_0402_1005Metric, F.Cu at (10.5, 18.0)
- added R_OP: 100k, Resistor_SMD:R_0402_1005Metric, F.Cu at (9.50, 11.0)
- added R_RA: 100k, Resistor_SMD:R_0402_1005Metric, F.Cu at (5.00, 18.0)
- added R_RL: 100k, Resistor_SMD:R_0402_1005Metric, F.Cu at (4.00, 17.5)
- added R_SCL: 4.7k, Resistor_SMD:R_0402_1005Metric, F.Cu at (19.0, 11.0)
- added R_SDA: 4.7k, Resistor_SMD:R_0402_1005Metric, F.Cu at (15.0, 11.0)
- added U1: MAX30102, custom:MAX30102EFDT, B.Cu at (7.50, 20.0)
- added U2: MAX30208, custom:MAX30208CLBT, B.Cu at (17.5, 20.0)
- added U3: AD8232, QFN-20-1EP_4x4mm_P0.5mm_EP2.6x2.6mm, F.Cu at (7.00, 15.0)
- added U4: ADS1115, Package_VSSOP:VSSOP-10_3x3mm_P0.5mm, F.Cu at (18.0, 15.0)
Routing:
- net OP_AP: track 0.00 -> 16.1 mm
- net HP_P1: track 0.00 -> 6.09 mm
- net HP_N1: track 0.00 -> 4.60 mm
- net GAIN_A: track 0.00 -> 4.56 mm
- net GAIN_B: track 0.00 -> 4.42 mm
- net RLDRIVE: track 0.00 -> 4.18 mm
- net VCC_3V3: track 0.00 -> 4.06 mm
- net RLDRIVE_IC: track 0.00 -> 3.08 mm
- net OP_AM: track 0.00 -> 1.50 mm
Other:
- board outline added: 25 x 25 mm
