File: board-a-main/board-a-main.kicad_pcb (KiCad board)
At the start: 2 copper layers, 0 parts

Commit message: session-2: board-a progress + board-b schematic updates
Co-Authored-By: Claude Sonnet 4.6 <noreply@anthropic.com>
Parts:
- added BOOT: SW_Push, Button_Switch_SMD:SW_Push_1P1T_NO_CK_KMR2, F.Cu at (205.2, 61.1)
- added C1: 10uF, Capacitor_SMD:C_0805_2012Metric, F.Cu at (201.5, 50.5)
- added C_BAT1: 10uF, Capacitor_SMD:C_0805_2012Metric, F.Cu at (198.0, 44.5)
- added C_BAT2: 100nF, Capacitor_SMD:C_0402_1005Metric, F.Cu at (198.0, 43.0)
- added C_BATT1: 100nF, Capacitor_SMD:C_0402_1005Metric, F.Cu at (192.3, 66.3)
- added C_Delay1: 1uF, Capacitor_SMD:C_0805_2012Metric, F.Cu at (208.9, 54.2)
- added C_IMU_DEC1: 100nF, Capacitor_SMD:C_0402_1005Metric, F.Cu at (194.0, 50.1)
- added C_LDO_IN1: 10uF, Capacitor_SMD:C_0805_2012Metric, F.Cu at (212.2, 40.3)
- added C_LDO_OUT1: 10uF, Capacitor_SMD:C_0805_2012Metric, F.Cu at (202.0, 36.5)
- added C_LDO_OUT2: 100nF, Capacitor_SMD:C_0402_1005Metric, F.Cu at (203.5, 39.0)
- added C_MCP_DEC1: 100nF, Capacitor_SMD:C_0402_1005Metric, F.Cu at (200.2, 34.0)
- added C_SHT_DEC1: 100nF, Capacitor_SMD:C_0402_1005Metric, F.Cu at (215.0, 59.5)
- added C_decoupling1: 100nF, Capacitor_SMD:C_0402_1005Metric, F.Cu at (189.6, 65.8)
- added C_decoupling2: 10uF, Capacitor_SMD:C_0805_2012Metric, F.Cu at (186.9, 66.1)
- added D1: PRTR5V0U2X, Package_TO_SOT_SMD:SOT-143, F.Cu at (199.6, 47.5)
- added D_LED_CHG1: RED, LED_SMD:LED_0402_1005Metric, F.Cu at (203.8, 34.0)
- added J1: USB_C_Receptacle_USB2.0_16P, Connector_USB:USB_C_Receptacle_GCT_USB4105-xx-A_16P_TopMnt_Horizontal, F.Cu at (212.2, 46.7)
- added J2: JST-SH 2-Pin, Connector_JST:JST_SH_SM02B-SRSS-TB_1x02-1MP_P1.00mm_Horizontal, B.Cu at (195.1, 64.1)
- added J3: Conn_01x10_Socket, 1_Global_Library:FPC-SMD_10P-P0.50_XUNPU_FPC-05F-10PH15, B.Cu at (186.7, 39.0)
- added J4: Conn_01x03, Connector_Wire:SolderWire-0.127sqmm_1x03_P3.7mm_D0.48mm_OD1mm, F.Cu at (201.0, 65.4)
- added J_DISP1: Conn_01x08, Connector_FFC-FPC:Hirose_FH12-8S-0.5SH_1x08-1MP_P0.50mm_Horizontal, F.Cu at (186.1, 44.9)
- added J_POGO_RLD1: Conn_01x01, TestPoint:TestPoint_Pad_D2.0mm, F.Cu at (183.9, 35.1)
- added R1: 4.3k, Resistor_SMD:R_0402_1005Metric, F.Cu at (204.9, 40.4)
- added REF1: MountingHole_2.1mm, MountingHole:MountingHole_2.1mm, F.Cu at (212.8, 35.8)
- added REF2: MountingHole_2.1mm, MountingHole:MountingHole_2.1mm, F.Cu at (212.8, 64.8)
- added RESET1: SW_Push, Button_Switch_SMD:SW_Push_1P1T_NO_CK_KMR2, F.Cu at (213.2, 55.0)
- added R_BATT_1: 100k, Resistor_SMD:R_0402_1005Metric, F.Cu at (193.3, 66.3)
- added R_BATT_2: 100k, Resistor_SMD:R_0402_1005Metric, F.Cu at (191.4, 66.3)
- added R_I2C_SCL1: 4.7k, Resistor_SMD:R_0402_1005Metric, F.Cu at (189.7, 33.4)
- added R_I2C_SDA1: 4.7k, Resistor_SMD:R_0402_1005Metric, F.Cu at (188.8, 34.8)
- added R_INT_PU1: 10k, Resistor_SMD:R_0402_1005Metric, F.Cu at (197.8, 66.2)
- added R_LED_CHG1: 1k, Resistor_SMD:R_0402_1005Metric, F.Cu at (205.9, 34.0)
- added R_MCP_RST1: 10k, Resistor_SMD:R_0402_1005Metric, F.Cu at (188.8, 37.7)
- added R_Pull_Up_ESP1: 10k, Resistor_SMD:R_0805_2012Metric, F.Cu at (204.1, 57.7)
- added R_Pull_Up_ESP2: 10k, Resistor_SMD:R_0805_2012Metric, F.Cu at (206.9, 54.2)
- added R_USB_CC1: 5.1k, Resistor_SMD:R_0402_1005Metric, F.Cu at (205.9, 48.5)
- added R_USB_CC2: 5.1k, Resistor_SMD:R_0402_1005Metric, F.Cu at (205.8, 45.4)
- added U1: ESP32-C3-MINI-1, custom:ESP32-C3-MINI-1, F.Cu at (189.5, 58.3)
- added U2: MCP73831-2-OT, Package_TO_SOT_SMD:SOT-23-5, F.Cu at (202.8, 42.5)
- added U3: AP2112K-3.3, Package_TO_SOT_SMD:SOT-23-5, F.Cu at (205.6, 36.5)
- added U4: USBLC6-2SC6, Package_TO_SOT_SMD:SOT-23-6, F.Cu at (203.3, 47.0)
- added U5: MCP23008-xSS, Package_SO:SSOP-20_5.3x7.2mm_P0.65mm, F.Cu at (194.5, 37.3)
- added U7: SHT30-DIS, Sensor_Humidity:Sensirion_DFN-8-1EP_2.5x2.5mm_P0.5mm_EP1.1x1.7mm, F.Cu at (212.4, 59.6)
Routing:
- net GND: track 0.00 -> 260.1 mm, vias 0 -> 17
- net +3.3V: track 0.00 -> 235.7 mm, vias 0 -> 7
- net +BATT: track 0.00 -> 113.7 mm, vias 0 -> 3
- net /I2C_SDA: track 0.00 -> 106.6 mm, vias 0 -> 2
- net /I2C_SCL: track 0.00 -> 87.1 mm, vias 0 -> 6
- net /INT_EXPANDER: track 0.00 -> 67.5 mm, vias 0 -> 2
- net /BTN_2: track 0.00 -> 62.9 mm, vias 0 -> 1
- net /ECG_SDN: track 0.00 -> 53.9 mm, vias 0 -> 1
- net /RESET_BTN: track 0.00 -> 53.8 mm, vias 0 -> 2
- net /BTN_1: track 0.00 -> 53.7 mm, vias 0 -> 1
- net /DISP_RST: track 0.00 -> 51.6 mm, vias 0 -> 2
- net VBUS: track 0.00 -> 42.9 mm
- net /ECG_LOD-: track 0.00 -> 42.3 mm, vias 0 -> 1
- net /DISP_CS: track 0.00 -> 40.3 mm, vias 0 -> 2
- net /DISP_BL: track 0.00 -> 35.0 mm, vias 0 -> 2
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- added copper zone on B.Cu, net GND
- added copper zone on F.Cu, net GND
Other:
- board outline added: 35.4 x 35.5 mm
