File: board-a-main/board-a-main.kicad_sch (KiCad schematic)
At the start: 0 parts

Commit message: session-2: board-a progress + board-b schematic updates
Co-Authored-By: Claude Sonnet 4.6 <noreply@anthropic.com>
Parts:
- added C1, C_BAT1, C_LDO_IN1, C_LDO_OUT1, C_decoupling2: 10uF, Capacitor_SMD:C_0805_2012Metric, symbol Device:C
- added C_BAT2, C_BATT1, C_LDO_OUT2, C_MCP_DEC1, C_SHT_DEC1, C_decoupling1: 100nF, Capacitor_SMD:C_0402_1005Metric, symbol Device:C
- added C_Delay1: 1uF, Capacitor_SMD:C_0805_2012Metric, symbol Device:C
- added D1: PRTR5V0U2X, Package_TO_SOT_SMD:SOT-143, symbol Power_Protection:PRTR5V0U2X
- added D_LED_CHG1: RED, LED_SMD:LED_0402_1005Metric, symbol Device:LED
- added J1: USB_C_Receptacle_USB2.0_16P, Connector_USB:USB_C_Receptacle_GCT_USB4105-xx-A_16P_TopMnt_Horizontal, symbol Connector:USB_C_Receptacle_USB2.0_16P
- added J2: JST-SH 2-Pin, Connector_JST:JST_SH_SM02B-SRSS-TB_1x02-1MP_P1.00mm_Horizontal, symbol Connector_Generic:Conn_01x02
- added J3: Conn_01x10_Socket, 1_Global_Library:FPC-SMD_10P-P0.50_XUNPU_FPC-05F-10PH15, symbol Connector:Conn_01x10_Socket
- added J4: Conn_01x03, Connector_Wire:SolderWire-0.127sqmm_1x03_P3.7mm_D0.48mm_OD1mm, symbol Connector_Generic:Conn_01x03
- added J_DISP1: Conn_01x08, Connector_FFC-FPC:Hirose_FH12-8S-0.5SH_1x08-1MP_P0.50mm_Horizontal, symbol Connector_Generic:Conn_01x08
- added J_POGO_RLD1: Conn_01x01, TestPoint:TestPoint_Pad_D2.0mm, symbol Connector_Generic:Conn_01x01
- added R1: 4.3k, Resistor_SMD:R_0402_1005Metric, symbol Device:R
- added RESET1, SW_BOOT1: SW_Push, Button_Switch_SMD:SW_Push_1P1T_NO_CK_KMR2, symbol Switch:SW_Push
- added R_BATT_1, R_BATT_2: 100k, Resistor_SMD:R_0402_1005Metric, symbol Device:R
- added R_I2C_SCL1, R_I2C_SDA1: 4.7k, Resistor_SMD:R_0402_1005Metric, symbol Device:R
- added R_INT_PU1, R_MCP_RST1: 10k, Resistor_SMD:R_0402_1005Metric, symbol Device:R
- added R_LED_CHG1: 1k, Resistor_SMD:R_0402_1005Metric, symbol Device:R
- added R_Pull_Up_ESP1, R_Pull_Up_ESP2: 10k, Resistor_SMD:R_0805_2012Metric, symbol Device:R
- added R_USB_CC1, R_USB_CC2: 5.1k, Resistor_SMD:R_0402_1005Metric, symbol Device:R
- added U1: ESP32-C3-MINI-1, custom:ESP32-C3-MINI-1, symbol Espressif:ESP32-C3-MINI-1
- added U2: MCP73831-2-OT, Package_TO_SOT_SMD:SOT-23-5, symbol Battery_Management:MCP73831-2-OT
- added U3: AP2112K-3.3, Package_TO_SOT_SMD:SOT-23-5, symbol Regulator_Linear:AP2112K-3.3
- added U4: USBLC6-2SC6, Package_TO_SOT_SMD:SOT-23-6, symbol Power_Protection:USBLC6-2SC6
- added U5: MCP23008-xSS, Package_SO:SSOP-20_5.3x7.2mm_P0.65mm, symbol Interface_Expansion:MCP23008-xSS
- added U7: SHT30-DIS, Sensor_Humidity:Sensirion_DFN-8-1EP_2.5x2.5mm_P0.5mm_EP1.1x1.7mm, symbol Sensor_Humidity:SHT30-DIS
Connections:
- new net: J1.A5 (CC1), R_USB_CC1.1
- new net: C_LDO_OUT1.1, C_LDO_OUT2.2, U3.5 (VOUT)
- new net: R1.2, U2.5 (PROG)
- new net: J1.A6 (D+), J1.B6 (D+), U4.1 (I/O1)
- new net: J1.A7 (D-), J1.B7 (D-), U4.3 (I/O2)
- new net: J1.B5 (CC2), R_USB_CC2.1
- new net: D_LED_CHG1.1 (K), R_LED_CHG1.2
- new net: R_MCP_RST1.2, U5.6 (~{RESET})
- new net +3.3V: C_LDO_OUT1.2, C_LDO_OUT2.1, C_MCP_DEC1.1, C_SHT_DEC1.2, C_decoupling1.1, C_decoupling2.1, J3.1 (Pin_1), J_DISP1.1 (Pin_1), R_I2C_SCL1.1, R_I2C_SDA1.2, R_INT_PU1.1, R_MCP_RST1.1, R_Pull_Up_ESP1.1, R_Pull_Up_ESP2.2, U1.3 (3V3), U5.20 (VDD), U7.5 (VDD), U7.6 (~{RESET})
- new net +BATT: C_BAT1.1, C_BAT2.1, C_LDO_IN1.2, J2.1 (Pin_1), R_BATT_1.1, U2.3 (V_{BAT}), U3.1 (VIN), U3.3 (EN)
- new net BATT_ADC: C_BATT1.1, R_BATT_1.2, R_BATT_2.1, U1.5 (GPIO2/ADC1_CH2)
- new net BOOT_BTN: R_Pull_Up_ESP1.2, SW_BOOT1.2, U1.23 (GPIO9)
- new net BTN_1: J4.2 (Pin_2), U5.12 (GP0)
- new net BTN_2: J4.3 (Pin_3), U5.13 (GP1)
- new net CHG_STAT: D_LED_CHG1.2 (A), U2.1 (STAT)
- new net DISP_BL: J_DISP1.8 (Pin_8), U1.6 (GPIO3/ADC1_CH3)
- new net DISP_CS: J_DISP1.3 (Pin_3), U1.16 (GPIO10)
- new net DISP_DC: J_DISP1.4 (Pin_4), U1.22 (GPIO8)
- new net DISP_RST: J_DISP1.5 (Pin_5), U5.17 (GP5)
- new net ECG_LOD+: J3.8 (Pin_8), U5.15 (GP3)
- new net ECG_LOD-: J3.7 (Pin_7), U5.16 (GP4)
- new net ECG_RLD_PAD: J3.9 (Pin_9), J_POGO_RLD1.1 (Pin_1)
- new net ECG_SDN: J3.6 (Pin_6), U1.31 (GPIO21/U0TXD)
- new net GND: C1.1, C_BAT1.2, C_BAT2.2, C_BATT1.2, C_Delay1.2, C_LDO_IN1.1, C_MCP_DEC1.2, C_SHT_DEC1.1, C_decoupling1.2, C_decoupling2.2, D1.1 (GND), J1.A1 (GND), J1.A12 (GND), J1.B1 (GND), J1.B12 (GND), J1.SH (SHIELD), J2.2 (Pin_2), J3.2 (Pin_2), J4.1 (Pin_1), J_DISP1.2 (Pin_2), R1.1, RESET1.2, R_BATT_2.2, R_USB_CC1.2, R_USB_CC2.2, SW_BOOT1.1, U1.1 (GND), U1.11 (GND), U1.14 (GND), U1.2 (GND), U1.36 (GND), U1.37 (GND), U1.38 (GND), U1.39 (GND), U1.40 (GND), U1.41 (GND), U1.42 (GND), U1.43 (GND), U1.44 (GND), U1.45 (GND), U1.46 (GND), U1.47 (GND), U1.48 (GND), U1.49 (GND), U1.50 (GND), U1.51 (GND), U1.52 (GND), U1.53 (GND), U2.2 (V_{SS}), U3.2 (GND), U4.2 (GND), U5.3 (A2), U5.4 (A1), U5.5 (A0), U5.9 (VSS), U7.2 (ADDR), U7.7 (R), U7.8 (VSS), U7.9 (VSS)
- new net I2C_SCL: J3.5 (Pin_5), R_I2C_SCL1.2, U1.19 (GPIO5/ADC2_CH0), U5.1 (SCL), U7.4 (SCL)
- new net I2C_SDA: J3.4 (Pin_4), R_I2C_SDA1.1, U1.18 (GPIO4/ADC1_CH4), U5.2 (SDA), U7.1 (SDA)
- new net INT_ADC: J3.3 (Pin_3), U5.19 (GP7)
- new net INT_EXPANDER: R_INT_PU1.2, U1.12 (GPIO0/ADC1_CH0/XTAL_32K_P), U5.8 (INT)
- new net INT_MAX: J3.10 (Pin_10), U5.18 (GP6)
- new net RESET_BTN: C_Delay1.1, RESET1.1, R_Pull_Up_ESP2.1, U1.8 (EN/CHIP_PU)
- new net SPI_MOSI: J_DISP1.6 (Pin_6), U1.20 (GPIO6)
- new net SPI_SCK: J_DISP1.7 (Pin_7), U1.21 (GPIO7)
- new net USB_D+: U1.27 (GPIO19/USB_D+), U4.6 (I/O1)
- new net USB_D-: U1.26 (GPIO18/USB_D-), U4.4 (I/O2)
- new net VBUS: C1.2, D1.4 (VCC), J1.A4 (VBUS), J1.A9 (VBUS), J1.B4 (VBUS), J1.B9 (VBUS), R_LED_CHG1.1, U2.4 (V_{DD}), U4.5 (VBUS)
- no-connect marks 0 -> 7
